File: UPS Raspberry.kicad_sch (KiCad schematic)
At the start: 20 parts, among them J1 Input +12V, J2 Buck converter, J3 Battery, K1 72mA, Q1 BC547, U1 LM317

Commit message: feat: updated circuit and docs
Parts:
- J1: value Input +12V -> 12V input
- J2: value Buck converter -> DC-DC output converter
- J3: value Battery -> 6V Pb Battery
- R1: value R -> 330
- R2: value R -> 1500
- R3: value R -> 100
- R4: value R -> 15
- gave numbers to parts that had none: 1
Changed lines of the file:
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@@
     (in_bom yes) (on_board yes)
     (property "Reference" "J3" (id 0) (at 128.27 64.77 0))
-    (property "Value" "Battery" (id 1) (at 128.27 67.31 0))
+    (property "Value" "6V Pb Battery" (id 1) (at 128.27 67.31 0))
     (property "Footprint" "" (id 2) (at 128.27 73.66 0)
       (effects (font (size 1.27 1.27)) hide)
@@
     (in_bom yes) (on_board yes)
     (property "Reference" "J1" (id 0) (at 201.93 63.5 0))
-    (property "Value" "Input +12V" (id 1) (at 200.66 66.04 0))
+    (property "Value" "12V input" (id 1) (at 200.66 66.04 0))
     (property "Footprint" "" (id 2) (at 198.12 60.96 0)
       (effects (font (size 1.27 1.27)) hide)
@@
       (effects (font (size 1.27 1.27)) (justify left))
     )
-    (property "Value" "R" (id 1) (at 122.428 95.123 0)
+    (property "Value" "330" (id 1) (at 122.428 95.123 0)
       (effects (font (size 1.27 1.27)) (justify left))
     )
@@
       (effects (font (size 1.27 1.27)) (justify left))
     )
-    (property "Value" "R" (id 1) (at 122.428 107.823 0)
+    (property "Value" "1500" (id 1) (at 122.428 107.823 0)
       (effects (font (size 1.27 1.27)) (justify left))
     )
@@
     )
     (property "Datasheet" "~" (id 3) (at 120.65 106.68 0)
-      (effects (font (size 1.27 1.27)) hide)
-    )
-    (pin "1")
-    (pin "2")
-  )
-  (symbol (lib_id "Device:R") (at 111.76 123.19 90) (unit 1)
-    (in_bom yes) (on_board yes)
-    (property "Reference" "R4" (id 0) (at 110.5916 121.412 0)
-      (effects (font (size 1.27 1.27)) (justify left))
-    )
-    (property "Value" "R" (id 1) (at 112.903 121.412 0)
-      (effects (font (size 1.27 1.27)) (justify left))
-    )
-    (property "Footprint" "" (id 2) (at 111.76 124.968 90)
-      (effects (font (size 1.27 1.27)) hide)
-    )
-    (property "Datasheet" "~" (id 3) (at 111.76 123.19 0)
-      (effects (font (size 1.27 1.27)) hide)
-    )
-    (pin "1")
-    (pin "2")
-  )
-  (symbol (lib_id "Device:R") (at 111.76 114.3 90) (unit 1)
-    (in_bom yes) (on_board yes)
-    (property "Reference" "R3" (id 0) (at 110.5916 112.522 0)
-      (effects (font (size 1.27 1.27)) (justify left))
-    )
-    (property "Value" "R" (id 1) (at 112.903 112.522 0)
-      (effects (font (size 1.27 1.27)) (justify left))
-    )
-    (property "Footprint" "" (id 2) (at 111.76 116.078 90)
-      (effects (font (size 1.27 1.27)) hide)
-    )
-    (property "Datasheet" "~" (id 3) (at 111.76 114.3 0)
       (effects (font (size 1.27 1.27)) hide)
     )
@@
       (effects (font (size 1.27 1.27)) (justify left))
     )
-    (property "Value" "Buck converter" (id 1) (at 200.152 90.1446 0)
+    (property "Value" "DC-DC output converter" (id 1) (at 200.152 90.1446 0)
       (effects (font (size 1.27 1.27)) (justify left))
     )
@@
   (symbol (lib_id "Transistor_FET:2N7000") (at 166.37 109.22 0) (unit 1)
     (in_bom yes) (on_board yes)
-    (property "Reference" "Q?" (id 0) (at 171.5516 108.0516 0)
+    (property "Reference" "Q2" (id 0) (at 171.5516 108.0516 0)
       (effects (font (size 1.27 1.27)) (justify left))
     )
@@
     )
     (pin "1")
+  )
+  (symbol (lib_id "Device:R") (at 111.76 114.3 90) (unit 1)
+    (in_bom yes) (on_board yes)
+    (property "Reference" "R3" (id 0) (at 111.76 109.22 90))
+    (property "Value" "100" (id 1) (at 111.76 111.76 90))
+    (property "Footprint" "" (id 2) (at 111.76 116.078 90)
+      (effects (font (size 1.27 1.27)) hide)
+    )
+    (property "Datasheet" "~" (id 3) (at 111.76 114.3 0)
+      (effects (font (size 1.27 1.27)) hide)
+    )
+    (pin "1")
+    (pin "2")
+  )
+  (symbol (lib_id "Device:R") (at 111.76 123.19 90) (unit 1)
+    (in_bom yes) (on_board yes)
+    (property "Reference" "R4" (id 0) (at 111.76 118.11 90))
+    (property "Value" "15" (id 1) (at 111.76 120.65 90))
+    (property "Footprint" "" (id 2) (at 111.76 124.968 90)
+      (effects (font (size 1.27 1.27)) hide)
+    )
+    (property "Datasheet" "~" (id 3) (at 111.76 123.19 0)
+      (effects (font (size 1.27 1.27)) hide)
+    )
+    (pin "1")
+    (pin "2")
   )
   (sheet_instances
@@
     )
     (path "/00000000-0000-0000-0000-000061aeb62f"
-      (reference "J1") (unit 1) (value "Input +12V") (footprint "")
+      (reference "J1") (unit 1) (value "12V input") (footprint "")
     )
     (path "/00000000-0000-0000-0000-000061b456ad"
-      (reference "J2") (unit 1) (value "Buck converter") (footprint "")
+      (reference "J2") (unit 1) (value "DC-DC output converter") (footprint "")
     )
     (path "/00000000-0000-0000-0000-000061abf0df"
-      (reference "J3") (unit 1) (value "Battery") (footprint "")
+      (reference "J3") (unit 1) (value "6V Pb Battery") (footprint "")
     )
     (path "/00000000-0000-0000-0000-000061ac2173"
@@
     )
     (path "/00000000-0000-0000-0000-000061b776e5"
-      (reference "Q?") (unit 1) (value "2N7000") (footprint "Package_TO_SOT_THT:TO-92_Inline")
+      (reference "Q2") (unit 1) (value "2N7000") (footprint "Package_TO_SOT_THT:TO-92_Inline")
     )
     (path "/00000000-0000-0000-0000-000061afa0ef"
-      (reference "R1") (unit 1) (value "R") (footprint "")
+      (reference "R1") (unit 1) (value "330") (footprint "")
     )
     (path "/00000000-0000-0000-0000-000061afadb3"
-      (reference "R2") (unit 1) (value "R") (footprint "")
-    )
-    (path "/00000000-0000-0000-0000-000061b007f3"
-      (reference "R3") (unit 1) (value "R") (footprint "")
-    )
-    (path "/00000000-0000-0000-0000-000061affcb5"
-      (reference "R4") (unit 1) (value "R") (footprint "")
+      (reference "R2") (unit 1) (value "1500") (footprint "")
+    )
+    (path "/6fa36bf6-d5ce-4ed2-820e-4046f04e8a6c"
+      (reference "R3") (unit 1) (value "100") (footprint "")
+    )
+    (path "/817aa12c-c5fe-4da1-8b21-8d07070bc989"
+      (reference "R4") (unit 1) (value "15") (footprint "")
     )
     (path "/00000000-0000-0000-0000-000061ac8c63"
